Commit message: Add 6-DoF MoveIt integration and documentation

File: src/lerobot_description/urdf/so101.urdf.xacro (robot description, xacro)
@@ -2,9 +2,9 @@
 <robot name="$(arg robot_name)" xmlns:xacro="http://www.ros.org/wiki/xacro">
     <xacro:arg name="robot_name" default="so101" />
-    <!-- Pass through for Gazebo: use MoveIt controller config when launching with MoveIt (kienmatics_controller) -->
+    <!-- Pass through for Gazebo: use MoveIt controller config when launching with MoveIt (kinematics_controller) -->
     <xacro:arg name="ros2_control_config_file" default="$(find lerobot_controller)/config/so101_controllers.yaml" />
     <xacro:arg name="use_sim" default="true" />
     <xacro:arg name="calibration_file" default="" />
-    <xacro:arg name="serial_port" default="/dev/ttyACM1" />
+    <xacro:arg name="serial_port" default="/dev/ttyACM0" />
     <xacro:include filename="$(find lerobot_description)/urdf/so101_new_calib.urdf" />
     <xacro:if value="$(arg use_sim)">

File: src/lerobot_description/urdf/so101_new_calib.urdf (robot description, URDF)
Before this commit: robot so101_new_calib, 9 links, 8 joints
Joints:
- joint elbow_rotate: limit lower=-1.38 upper=1.38 effort=10 velocity=10 -> lower=-1.80 upper=1.94 effort=10 velocity=10
- joint shoulder_lift: limit lower=-1.74533 upper=1.74533 effort=10 velocity=10 -> lower=-1.75 upper=2.05 effort=10 velocity=10
- joint shoulder_pan: limit lower=-1.91986 upper=1.91986 effort=10 velocity=10 -> lower=-1.95 upper=2.25 effort=10 velocity=10
- joint wrist_flex: limit lower=-1.65806 upper=1.65806 effort=10 velocity=10 -> lower=-1.93 upper=1.76 effort=10 velocity=10

File: src/lerobot_description/urdf/so101_ros2_control.xacro (robot description, xacro)
@@ -30,4 +30,12 @@
             <state_interface name="velocity"/>
         </joint>
+        <joint name="elbow_rotate">
+            <command_interface name="position">
+                <param name="min">-1.38</param>
+                <param name="max">1.38</param>
+            </command_interface>
+            <state_interface name="position"/>
+            <state_interface name="velocity"/>
+        </joint>
         <joint name="wrist_flex">
             <command_interface name="position">

File: src/lerobot_description/urdf/so101_ros2_control_real.xacro (robot description, xacro)
@@ -23,4 +23,8 @@
       <state_interface name="position"/>
     </joint>
+    <joint name="elbow_rotate">
+      <command_interface name="position"/>
+      <state_interface name="position"/>
+    </joint>
     <joint name="wrist_flex">
       <command_interface name="position"/>

File: src/lerobot_moveit/config/so101_new_calib.ros2_control.xacro (robot description, xacro)
@@ -38,4 +38,14 @@
                 <state_interface name="effort"/>
             </joint>
+            <joint name="elbow_rotate">
+                <command_interface name="position"/>
+                <command_interface name="velocity"/>
+                <command_interface name="effort"/>
+                <state_interface name="position">
+                  <param name="initial_value">${initial_positions['elbow_rotate']}</param>
+                </state_interface>
+                <state_interface name="velocity"/>
+                <state_interface name="effort"/>
+            </joint>
             <joint name="wrist_flex">
                 <command_interface name="position"/>
