Commit message: Add : 6 Joint URDF

File: src/lerobot_description/urdf/so101_new_calib.urdf (robot description, URDF)
Before this commit: robot so101_new_calib, 8 links, 7 joints
Links:
- added link link5_link, mass 0.05; collision mesh filename=package://lerobot_description/meshes/so101/link5.stl scale=0.001 0.001 0.001; collision mesh filename=package://lerobot_description/meshes/so101/motor_holder_so1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
- link lower_arm_link: geometry collision mesh filename=package://lerobot_description/meshes/so101/LINK4.stl scale=0.001 0.001 0.001; visual mesh filename=package://lerobot_description/meshes/so101/LINK4.stl scale=0.001 0.001 0.001
Joints:
- added joint elbow_rotate: type revolute, parent lower_arm_link, child link5_link, origin xyz=0 0 0.0143 rpy=0 0 0, axis 1 0 0, limit lower=-1.38 upper=1.38 effort=10 velocity=10
- joint wrist_flex: origin xyz=-0.1349 0.0052 3.62355e-17 rpy=4.02456e-15 8.67362e-16 -1.5708 -> xyz=-0.1349 0.0052 -0.0143 rpy=4.02456e-15 8.67362e-16 -1.5708; parent lower_arm_link -> link5_link

Commit message: Add : EEF frame link

File: src/lerobot_description/urdf/so101_new_calib.urdf (robot description, URDF)
Before this commit: robot so101_new_calib, 9 links, 8 joints
Links:
- added link eef_frame_link, mass 1e-9
Joints:
- added joint eef_frame_joint: type fixed, parent gripper_link, child eef_frame_link, origin xyz=0 0 -0.0981274 rpy=0 3.14159 0
